Commit message: Added new models for training. TODO: Check and see if can revolute joints.

File: models/poc.urdf (robot description, URDF)
Before this commit: robot cart, 1 links, 0 joints
Links:
- link baseLink: geometry collision box size=0.2 0.2 0.05; visual box size=0.03 0.03 0.03

File: models/uav_fluid.urdf (robot description, URDF)
Before this commit: robot uav, 2 links, 1 joints
Links:
- link uavLink: geometry collision box size=0.2 0.2 0.03; visual box size=0.2 0.2 0.05

Commit message: Added new models for training. TODO: Check and see if can revolute joints.

File: models/poc.urdf (robot description, URDF)
Before this commit: robot cart, 1 links, 0 joints
Links:
- link baseLink: mass 1 -> 1.5; geometry collision box size=0.2 0.2 0.05; visual box size=0.1 0.1 0.05

File: models/uav_fluid.urdf (robot description, URDF)
Before this commit: robot uav, 2 links, 1 joints
Links:
- link fluidLink: mass 5 -> 2
- link uavLink: mass 1 -> 10
